File: Project Architecture.kicad_sch (KiCad schematic)
At the start: 0 parts

Commit message: Draft: The schematic update in the draft version
Other:
- removed sheet Section A - Title A
- removed sheet Section B - Title B
- added sheet Connectors (Connectors.kicad_sch)
- added sheet Holes, Fiducials (Holes, Fiducials.kicad_sch)
- added sheet IMU (IMU.kicad_sch)
- added sheet MCU (MCU.kicad_sch)
- note added: "Page 6"
- note added: "Page 7"
