File: 01_HAT_INA226.kicad_pcb (KiCad board)
At the start: 6 copper layers, 0 parts

Commit message: Fix: schematic
Parts:
- added C1: 100n X7R 50V, 0_capacitor_smd:C_0402_1005_DensityHigh, F.Cu at (167.0, 100.1)
- added C10: 3.9pF, Capacitor_SMD:C_0402_1005Metric, F.Cu at (140.1, 110.6)
- added C11: 100n X7R 50V, 0_capacitor_smd:C_0402_1005_DensityHigh, F.Cu at (155.2, 83.5)
- added C12: 100n X7R 50V, 0_capacitor_smd:C_0402_1005_DensityHigh, F.Cu at (155.2, 85.3)
- added C13: 100n X7R 50V, 0_capacitor_smd:C_0402_1005_DensityHigh, F.Cu at (155.2, 87.1)
- added C14: 1u X7R 10V, 0_capacitor_smd:C_0402_1005_DensityHigh, F.Cu at (155.2, 88.9)
- added C15: 4u7 X5R 25V, 0_capacitor_smd:C_0402_1005_DensityHigh, F.Cu at (157.8, 83.5)
- added C16: 100n X7R 50V, 0_capacitor_smd:C_0402_1005_DensityHigh, F.Cu at (157.8, 85.3)
- added C17: 1u X7R 10V, 0_capacitor_smd:C_0402_1005_DensityHigh, F.Cu at (157.8, 87.1)
- added C18: 100n X7R 50V, 0_capacitor_smd:C_0402_1005_DensityHigh, F.Cu at (157.8, 88.9)
- added C19: 100n X7R 50V, 0_capacitor_smd:C_0402_1005_DensityHigh, F.Cu at (160.4, 83.5)
- added C2: 100n X7R 50V, 0_capacitor_smd:C_0402_1005_DensityHigh, F.Cu at (167.0, 101.9)
- added C3: 1u X7R 25V, 0_capacitor_smd:C_0603_1608_DensityHigh, F.Cu at (167.4, 105.8)
- added C4: 10n X7R 100V, 0_capacitor_smd:C_0402_1005_DensityHigh, F.Cu at (167.0, 103.7)
- added C5: 4u7 X7R 16V, 0_capacitor_smd:C_0603_1608_DensityHigh, F.Cu at (167.4, 108.0)
- added C6: 100n X7R 50V, 0_capacitor_smd:C_0402_1005_DensityHigh, F.Cu at (135.8, 102.8)
- added C7: 100n X7R 50V, 0_capacitor_smd:C_0402_1005_DensityHigh, F.Cu at (135.8, 104.6)
- added C8: 100n X7R 50V, 0_capacitor_smd:C_0402_1005_DensityHigh, F.Cu at (135.8, 106.4)
- added C9: 3.9pF, Capacitor_SMD:C_0402_1005Metric, F.Cu at (140.1, 108.6)
- added FD1: Fiducial, 0_fiducials:Fiducial_1mm_Mask2mm, F.Cu at (144.0, 69.7)
- added FD2: Fiducial, 0_fiducials:Fiducial_1mm_Mask2mm, F.Cu at (144.0, 72.8)
- added FD3: Fiducial, 0_fiducials:Fiducial_1mm_Mask2mm, F.Cu at (147.2, 69.7)
- added FD4: Fiducial, 0_fiducials:Fiducial_1mm_Mask2mm, F.Cu at (147.2, 72.8)
- added FD5: Fiducial, 0_fiducials:Fiducial_1mm_Mask2mm, F.Cu at (150.3, 69.7)
- added FD6: Fiducial, 0_fiducials:Fiducial_1mm_Mask2mm, F.Cu at (150.3, 72.8)
- added H1: M3, MountingHole:MountingHole_3.2mm_M3_Pad, F.Cu at (138.4, 72.1)
- added H2: M3, MountingHole:MountingHole_3.2mm_M3_Pad, F.Cu at (138.4, 80.0)
- added H3: M3, MountingHole:MountingHole_3.2mm_M3_Pad, F.Cu at (138.4, 88.0)
- added H4: M3, MountingHole:MountingHole_3.2mm_M3_Pad, F.Cu at (138.4, 96.0)
- added J1: SM05B-GHS-TB, 0_connectors:JST_GH_SM05B-GHS-TB_1x05-1MP_P1.25mm_Horizontal, F.Cu at (159.8, 95.5)
- added J2: S2B-PH-SM4-TB, 0_connectors:JST_PH_S2B-PH-SM4-TB_1x02-1MP_P2.00mm_Horizontal, F.Cu at (159.0, 104.8)
- added R1: 10k 1%, 0_resistor_smd:R_0402_1005_DensityHigh, F.Cu at (135.8, 108.2)
- added R2: 10k 1%, 0_resistor_smd:R_0402_1005_DensityHigh, F.Cu at (135.8, 110.0)
- added R3: 10k 1%, 0_resistor_smd:R_0402_1005_DensityHigh, F.Cu at (135.8, 111.8)
- added R4: 10k 1%, 0_resistor_smd:R_0402_1005_DensityHigh, F.Cu at (135.8, 113.6)
- added R5: 2k 1%, 0_resistor_smd:R_0402_1005_DensityHigh, F.Cu at (160.4, 85.3)
- added R6: 2k 1%, 0_resistor_smd:R_0402_1005_DensityHigh, F.Cu at (160.4, 87.1)
- added TP1: TestPoint, 0_testpoint:TestPoint_Pad_D0.5mm, F.Cu at (164.9, 100.0)
- added TP2: TestPoint, 0_testpoint:TestPoint_Pad_D0.5mm, F.Cu at (164.9, 101.6)
- added TP3: TestPoint, 0_testpoint:TestPoint_Pad_D0.5mm, F.Cu at (164.9, 103.1)
- added TP4: TestPoint, 0_testpoint:TestPoint_Pad_D0.5mm, F.Cu at (164.9, 104.7)
- added TP5: TestPoint, 0_testpoint:TestPoint_Pad_D0.5mm, F.Cu at (164.9, 106.2)
- added TP6: TestPoint, 0_testpoint:TestPoint_Pad_D0.5mm, F.Cu at (137.9, 102.7)
- added TP7: TestPoint, 0_testpoint:TestPoint_Pad_D0.5mm, F.Cu at (137.9, 104.3)
- added TP8: TestPoint, 0_testpoint:TestPoint_Pad_D0.5mm, F.Cu at (137.9, 105.8)
- added TP9: TestPoint, 0_testpoint:TestPoint_Pad_D0.5mm, F.Cu at (137.9, 107.4)
- added U1: LP2992IM5-3.3/NOPB, Package_TO_SOT_SMD:SOT-23-5, F.Cu at (168.2, 94.2)
- added U2: BNO055, Package_LGA:LGA-28_5.2x3.8mm_P0.5mm, F.Cu at (142.2, 104.8)
- added U3: STM32G474RET3, 0_package_QFP:LQFP-64_10x10mm_P0.5mm, F.Cu at (161.1, 75.3)
- added Y1: ECS-.327-7-12-C-TR9, Crystal:Crystal_SMD_2012-2Pin_2.0x1.2mm, F.Cu at (143.5, 109.2)

Commit message: [PCB] Board outline Prelimary version]
Other:
- board outline added: 38.5 x 48.5 mm
Changed lines of the file:
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@@
+	)
+	(gr_rect
+		(start 133 66.5)
+		(end 171.5 115)
+		(stroke
+			(width 0.1)
+			(type solid)
+		)
+		(fill no)
+		(layer "Edge.Cuts")
 	)
 	(gr_rect
